File: Nano-CAN-Sense-HAT_Board/Nano-CAN-Sense-HAT.kicad_sch (KiCad schematic)
At the start: 33 parts, among them J1 Analog, J2 Digital, J3 Conn_02x04_Counter_Clockwise, J4 Conn_02x04_Counter_Clockwise, J5 Conn_01x05, J6 Conn_01x03, SW1 SW_Push, SW2 SW_Push, U1 LMC6484, U4 TCAN1044A

Commit message: added pdf and Screenshots
Other:
- note removed: "check footprints and define product. Add decoupling caps everywhere"
- note removed: "connector Footprint needs to be defined!"
Changed lines of the file:
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@@
-		)
-	)
-	(text "check footprints and define product.\nAdd decoupling caps everywhere"
-		(exclude_from_sim no)
-		(at 50.8 22.352 0)
-		(effects
-			(font
-				(size 4 4)
-			)
-			(justify left)
 		)
 	)
@@
 		)
 	)
-	(text "connector Footprint\nneeds to be defined!\n"
-		(exclude_from_sim no)
-		(at 222.758 25.4 0)
-		(effects
-			(font
-				(size 3 3)
-			)
-			(justify left)
-		)
-	)
