File: Nano-CAN-Sense-HAT_Board/Nano-CAN-Sense-HAT.kicad_sch (KiCad schematic)
At the start: 46 parts, among them J1 Analog, J2 Digital, J3 Conn_02x04_Counter_Clockwise, J4 Conn_02x04_Counter_Clockwise, J5 Conn_01x05, J6 Conn_01x03, SW1 SW_Push, SW2 SW_Push, U1 NCS20074DTB, U2 MCP2518FD-xQBB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

Commit message: Improved lables, better 5V protection diode, new images
Parts:
- added D6: D_Zener_5.1V, Diode_SMD:D_SOD-323, symbol Device:D_Zener
Connections:
- net +5V: now also D6.1 (K)
- net GND: now also D6.2 (A)
